Commit message: second update

File: myfirstrobot_description/urdf/myfirstrobot.urdf (robot description, URDF)
Before this commit: robot myfirstrobot, 2 links, 1 joints
Links:
- added link floor_link
- link base_link: geometry visual mesh filename=package://myfirstrobot_description/meshes/one2.stl
- link head_link: geometry visual mesh filename=package://myfirstrobot_description/meshes/one1.stl
Joints:
- added joint floor_to_base_joint: type fixed, parent floor_link, child base_link, origin xyz=0 0 0 rpy=0 0 0, axis 0 0 1
- joint servo_joint: axis 1 0 0 -> 0.1 0 0; limit lower=${-170 * M_PI / 180} upper=${170 * M_PI / 180} effort=176 -> lower=-0.5 upper=0.5 effort=0.1 velocity=0.1; origin xyz=0 0 0.5 -> xyz=0 0 0; type fixed -> revolute

Commit message: first commit

File: myfirstrobot_description/urdf/myfirstrobot.urdf (robot description, URDF)
Before this commit: robot myfirstrobot, 3 links, 2 joints
Links:
- link base_link: geometry collision mesh filename=package://myfirstrobot_description/meshes/xcollisionone2.stl; visual mesh filename=package://myfirstrobot_description/meshes/one2.stl
- link head_link: geometry collision mesh filename=package://myfirstrobot_description/meshes/xcollisionone1.stl; visual mesh filename=package://myfirstrobot_description/meshes/one1.stl
Joints:
- joint servo_joint: origin xyz=0 0 0 -> xyz=0 0 7.5
